File: PCB/Adalyn.sch (KiCad schematic (older format))
At the start: 73 parts, among them SW1 SW_Push, U101 ATmega32U4-A, U102 PRTR5V0U2X, Y1 16MHz

Commit message: NOT FINSIHED, first commit
Parts:
- removed C1: .1uF, Capacitor_SMD:C_0603_1608Metric_Pad1.08x0.95mm_HandSolder, symbol Device:C_Small
- removed U101: ATmega32U4-A, Package_QFP:TQFP-44_10x10mm_P0.8mm, symbol MCU_Microchip_ATmega:ATmega32U4-A
- added U1: ATmega32U2-AU, Package_QFP:TQFP-32_7x7mm_P0.8mm, symbol MCU_Microchip_ATmega:ATmega32U2-AU
- MX1, MX10, MX11, MX12, MX13, MX15, MX16, MX17, MX18, MX19, MX2, MX20, MX21, MX22, MX23, MX24, MX25, MX26, MX27, MX28, MX29, MX3, MX30, MX32, MX33, MX34, MX35, MX36, MX37, MX38, MX4, MX5, MX6, MX7, MX8, MX9: symbol MX_Alps_Hybrid:MX-NoLED -> Adalyn-rescue:MX-NoLED-MX_Alps_Hybrid
- U102: symbol keebio:PRTR5V0U2X -> Adalyn-rescue:PRTR5V0U2X-keebio
- USB101: symbol keebio:HRO-TYPE-C-31-M-12 -> Adalyn-rescue:HRO-TYPE-C-31-M-12-keebio
- Y1: footprint Crystal:Resonator_SMD_Murata_CSTxExxV-3Pin_3.0x1.1mm_HandSoldering -> Crystal:Resonator_SMD_muRata_CSTxExxV-3Pin_3.0x1.1mm
Connections:
- net +5V: now also U1.31 (UVCC), U1.32 (AVCC), U1.4 (VCC)
- net GND: now also U1.28 (UGND), U1.3 (GND)
- net at R4.2, SW1.2: now also U1.24 (PC1/~RESET)
- net at Y1.1: now also U1.1 (XTAL1)
- net at Y1.3: now also U1.2 (PC0/XTAL2)
- net at R5.1: now also U1.13 (~HWB~/PD7)
- net at R2.1: now also U1.29 (D+)
- net at R3.1: now also U1.30 (D-)
- net at C6.1: now also U1.27 (UCAP)
- no-connect marks 6 -> 4
Other:
- moved on the sheet: C6, R2, R3, R4, R5, SW1, Y1
