File: PCB/Adalyn.kicad_pcb (KiCad board)
At the start: 2 copper layers, 217.7 x 85.3 mm, 76 parts, among them SW1 SW_Push, U101 ATmega32U4-A, U102 PRTR5V0U2X, Y1 16MHz

Commit message: NOT FINSIHED, first commit
Parts:
- removed C1: .1uF, Capacitor_SMD:C_0603_1608Metric_Pad1.08x0.95mm_HandSolder
- removed G***: LOGO, Adalyn:Adalyn
- removed G***: LOGO, Adalyn:credit
- removed G***: LOGO, Adalyn:logo
- removed U101: ATmega32U4-A, Package_QFP:TQFP-44_10x10mm_P0.8mm
- added U1: ATmega32U2-AU, Package_QFP:TQFP-32_7x7mm_P0.8mm, B.Cu at (144.9, 86.2)
- Y1: footprint Crystal:Resonator_SMD_Murata_CSTxExxV-3Pin_3.0x1.1mm_HandSoldering -> Crystal:Resonator_SMD_muRata_CSTxExxV-3Pin_3.0x1.1mm
- moved D116 107.8 mm to (109.6, 12.2)
- moved D118 78.1 mm to (141.0, 18.9)
- moved D108 56.0 mm to (130.0, 21.1)
- moved D103 42.6 mm to (131.0, 14.7)
- moved SW1 23.4 mm to (145.6, 102.0), turned to 270 degrees
- moved Y1 19.1 mm to (152.4, 83.8), turned to 270 degrees
- moved R2 18.7 mm to (144.9, 78.1), turned to 90 degrees
- moved R5 18.4 mm to (144.5, 93.5), turned to 270 degrees
- moved C6 18.2 mm to (143.4, 78.1), turned to 90 degrees
- moved R3 16.5 mm to (146.4, 78.1), turned to 90 degrees
- moved C2 15.2 mm to (152.4, 86.6), turned to 0 degrees
- moved R102 12.6 mm to (148.4, 63.5)
- moved C5 12.6 mm to (147.9, 78.1), turned to 90 degrees
- moved L101 12.2 mm to (141.4, 63.5)
- moved R4 10.6 mm to (137.1, 83.5), turned to 0 degrees
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Routing:
- net ROW0: track 211.9 -> 0.00 mm, vias 2 -> 0
- net ROW3: track 211.7 -> 0.00 mm, vias 2 -> 0
- net ROW1: track 193.1 -> 0.00 mm, vias 2 -> 0
- net ROW2: track 184.3 -> 0.00 mm
- net Col0: track 176.8 -> 0.00 mm
- net Col1: track 164.5 -> 0.00 mm
- net Col9: track 161.3 -> 0.00 mm
- net Col3: track 123.3 -> 0.00 mm
- net Col7: track 123.1 -> 0.00 mm
- net Col8: track 123.0 -> 0.00 mm
- net Col2: track 120.4 -> 0.00 mm
- net Col6: track 109.0 -> 0.00 mm
- net GND: track 106.1 -> 17.1 mm, vias 11 -> 2
- net +5V: track 102.5 -> 14.3 mm, vias 8 -> 0
- net Col4: track 82.1 -> 0.00 mm
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- added copper zone on F.Cu, net GND

Commit message: update to 5.99
Other:
- net class Default removed

Commit message: puuuush
Changed lines of the file:
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@@
   (segment (start 152.396992 82.624349) (end 151.096992 82.624349) (width 0.25) (layer "B.Cu") (net 87))
   (segment (start 149.111513 83.407383) (end 150.313958 83.407383) (width 0.25) (layer "B.Cu") (net 87))
-  (zone (net 53) (net_name "GND") (layer "F.Cu") (hatch edge 0.508)
+  (zone (net 53) (net_name "GND") (layers F&B.Cu) (hatch edge 0.508)
     (connect_pads (clearance 0.508))
-    (min_thickness 0.254)
+    (min_thickness 0.254) (filled_areas_thickness no)
     (fill yes (thermal_gap 0.508) (thermal_bridge_width 0.508))
     (polygon
-      (pts
-        (xy 279.104099 141.470796)
-        (xy 17.604099 140.470796)
-        (xy 18.354099 25.220796)
-        (xy 273.854099 25.220796)
-      )
-    )
-  )
-  (zone (net 53) (net_name "GND") (layer "B.Cu") (hatch edge 0.508)
-    (connect_pads (clearance 0.508))
-    (min_thickness 0.254)
-    (fill yes (thermal_gap 0.508) (thermal_bridge_width 0.508))
-    (polygon
