File: PCB/Adalyn.kicad_sch (KiCad schematic)
At the start: 72 parts, among them SW1 SW_Push, U1 ATmega32U2-AU, U102 PRTR5V0U2X, Y1 16MHz

Commit message: initial commit: updated bom,pos, finished routing
Parts:
- removed U102: PRTR5V0U2X, Package_TO_SOT_SMD:SOT-143, symbol Adalyn-rescue:PRTR5V0U2X-keebio
- removed Y1: 16MHz, Crystal:Resonator_SMD_muRata_CSTxExxV-3Pin_3.0x1.1mm, symbol Device:Resonator_Small
- added C7, C8: 22pf, Capacitor_SMD:C_0805_2012Metric, symbol Device:C
- added U102: SRV05-4, Package_TO_SOT_SMD:SOT-23-6, symbol Power_Protection:SRV05-4
- added Y1: Crystal_GND24_Small, Crystal:Crystal_SMD_3225-4Pin_3.2x2.5mm, symbol Device:Crystal_GND24_Small
- C101, C2, C4: footprint Capacitor_SMD:C_0603_1608Metric_Pad1.08x0.95mm_HandSolder -> Capacitor_SMD:C_0805_2012Metric; LCSC (none) -> C49678
- C5: footprint Capacitor_SMD:C_0603_1608Metric_Pad1.08x0.95mm_HandSolder -> Capacitor_SMD:C_0805_2012Metric; LCSC (none) -> C91245
- C6: footprint Capacitor_SMD:C_0603_1608Metric_Pad1.08x0.95mm_HandSolder -> Capacitor_SMD:C_0805_2012Metric; LCSC (none) -> C28323
- D101, D102, D103, D104, D105, D106, D107, D108, D109, D110, D111, D112, D113, D114, D115, D116, D117, D118: LCSC (none) -> C68978
- F101: value 700mA -> Polyfuse; footprint Fuse:Fuse_0603_1608Metric -> Fuse:Fuse_1206_3216Metric; LCSC (none) -> C69688
- MX1, MX10, MX11, MX12, MX13, MX15, MX16, MX17, MX18, MX19, MX2, MX20, MX21, MX22, MX23, MX24, MX25, MX26, MX27, MX28, MX29, MX3, MX30, MX32, MX33, MX34, MX35, MX36, MX37, MX38, MX4, MX5, MX6, MX7, MX8, MX9: footprint MX_Only:MXOnly-1U-NoLED -> marbastlib-mx:SW_MX_1u
- R101, R102: footprint Resistor_SMD:R_0603_1608Metric -> Resistor_SMD:R_0805_2012Metric; LCSC (none) -> C27834
- R2, R3: footprint Resistor_SMD:R_0603_1608Metric_Pad0.98x0.95mm_HandSolder -> Resistor_SMD:R_0805_2012Metric; LCSC (none) -> C17561
- R4, R5: footprint Resistor_SMD:R_0603_1608Metric_Pad0.98x0.95mm_HandSolder -> Resistor_SMD:R_0805_2012Metric; LCSC (none) -> C17414
- SW1: LCSC (none) -> C318884
- U1: LCSC (none) -> C618733
- USB101: LCSC (none) -> C165948
Connections:
- net +5V: now also U102.5 (VP)
- net Col0: now also U1.16 (PB2)
- net Col1: now also U1.17 (PB3)
- net Col2: now also U1.18 (PB4)
- net Col3: now also U1.19 (PB5)
- net Col4: now also U1.20 (PB6)
- net Col5: now also U1.5 (PC2)
- net Col6: now also U1.6 (PD0)
- net Col7: now also U1.7 (PD1)
- net Col8: now also U1.8 (PD2)
- net Col9: now also U1.9 (PD3)
- net D+: now also U102.1 (IO1)
- net D-: now also U102.4 (IO3)
- net GND: now also C7.1, C8.1, U102.2 (VN), Y1.2, Y1.4
- net ROW0: now also U1.12 (PD6)
- net ROW1: now also U1.11 (PD5)
- net ROW2: now also U1.14 (PB0)
- net ROW3: now also U1.15 (PB1)
- net at MX1.2 (ROW): now also D101.2 (A); no longer D101.1 (A)
- net at MX4.2 (ROW): now also D101.1 (A); no longer D101.2 (A)
- net at MX7.2 (ROW): now also D102.2 (A); no longer D102.1 (A)
- net at MX11.2 (ROW): now also D102.1 (A); no longer D102.2 (A)
- net at MX16.2 (ROW): now also D103.2 (A); no longer D103.1 (A)
- net at MX20.2 (ROW): now also D103.1 (A); no longer D103.2 (A)
- net at MX23.2 (ROW): now also D104.2 (A); no longer D104.1 (A)
- net at MX27.2 (ROW): now also D104.1 (A); no longer D104.2 (A)
- net at MX32.2 (ROW): now also D105.2 (A); no longer D105.1 (A)
- net at MX36.2 (ROW): now also D105.1 (A); no longer D105.2 (A)
- net at MX3.2 (ROW): now also D111.2 (A); no longer D111.1 (A)
- net at MX6.2 (ROW): now also D111.1 (A); no longer D111.2 (A)
- net at MX9.2 (ROW): now also D112.2 (A); no longer D112.1 (A)
- net at MX13.2 (ROW): now also D112.1 (A); no longer D112.2 (A)
- net at MX18.2 (ROW): now also D118.2 (A); no longer D118.1 (A)
- net at MX22.2 (ROW): now also D118.1 (A); no longer D118.2 (A)
- net at MX25.2 (ROW): now also D113.2 (A); no longer D113.1 (A)
- net at MX29.2 (ROW): now also D113.1 (A); no longer D113.2 (A)
- net at MX34.2 (ROW): now also D114.2 (A); no longer D114.1 (A)
- net at MX38.2 (ROW): now also D114.1 (A); no longer D114.2 (A)
- net at U1.1 (XTAL1): now also C8.2, Y1.1
- net at U1.2 (PC0/XTAL2): now also C7.2, Y1.3
- no-connect marks 4 -> 6
Other:
- moved on the sheet: R2
